Commit message: add a robot

File: robots/aliengo_description/xacro/robot.xacro (robot description, xacro)
@@ -35,5 +35,5 @@
                 <mesh filename="package://aliengo_description/meshes/trunk.dae" scale="1 1 1"/>
             </geometry>
-            <material name="orange"/>
+            <material name="black"/>
         </visual>
         <collision>
